Commit message: Add imu_link tf

File: src/ired_bringup/urdf/ired.urdf.xacro (robot description, xacro)
@@ -11,4 +11,5 @@
     <link name="aruco_camera_link"/>
     <link name="base_cartesian_link"/>
+    <link name="imu_link"/>
     <!-- Base Joint (Projects ground reference to chassis center) -->
     <joint name="base_joint" type="fixed">
@@ -17,4 +18,11 @@
         <!-- Z = Elevation from ground to base_link origin (e.g., 0.05 m wheel radius) -->
         <origin xyz="0.0 0.0 0.65" rpy="0.0 0.0 0.0"/>
+    </joint>
+    <!-- IMU Sensor Joint -->
+    <joint name="imu_joint" type="fixed">
+        <parent link="base_link"/>
+        <child link="imu_link"/>
+        <!-- Adjust to match the physical IMU mounting position -->
+        <origin xyz="0.0 0.0 0.0" rpy="0.0 0.0 0.0"/>
     </joint>
     <!-- LiDAR Sensor Joint -->

Commit message: Change imu_link parent

File: src/ired_bringup/urdf/ired.urdf.xacro (robot description, xacro)
@@ -21,5 +21,5 @@
     <!-- IMU Sensor Joint -->
     <joint name="imu_joint" type="fixed">
-        <parent link="base_link"/>
+        <parent link="base_footprint"/>
         <child link="imu_link"/>
         <!-- Adjust to match the physical IMU mounting position -->
